File: hardware/P300_Arduino_IF/P300_Arduino_IF.sch (KiCad schematic (older format))
At the start: 28 parts, among them J1 Relay brd, J10 Pressure, J11 TGS2600, J12 I2C, J13 CO2, J14 5V, J2 DHT1, J3 DHT2, J4 Fan control, J5 TEMP1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

Commit message: Update der Platinen auf 0.23-dev
Änderungen von 0.22 zu 0.23 - P300_Arduino_IF
 - Linke Seite der Platine vergrößert auf ArduinoMega-Größe
 - Stecker für Displayanschluß ergänzt
 - Fünf weitere Bohrungen für Befestigung ergänzt
 - Leiterbahnen im größeren Abstand zu Durchbohrungen und Bauteilen verlegt
 - Connector für J12 I2C nach links verschoben, damit ausreichend Platz für JTS Stecker
 - Auf dem Stecker J4 sind die beiden Lüfteranschlüsse Lüfter 1 und Lüfter 2 getauscht. Damit ist der Stecker kompatibel zu Pluggit. Der Pluggit-Lüfter-Steuerstecker kann direkt aufgesteckt werden, wenn Molex Stiftleiste - KK - 1x8-polig - Stecker, Molex-Best-Nr. 22272081 verwendet wird.

Änderungen von 0.22 zu 0.23 - P300_HiVolt
 - 230V Lüfteranschluss kompatibel zu Pluggit, Molex Stiftleiste - Mini-Fit Jr - 2x4-polig - Stecker, Molex-Best-Nr. 39281083
 - Stecker J3, J4 für Relais auf Molex Stiftleiste - Mini-Fit Jr - 2x3-polig - Stecker, Molex-Best-Nr. 39288060 geändert.
 - Änderung der Belegung der Stecker J3, J4 für die Verwendung es Relaisboards mit den Ralaisanschlüssen: Mitte = Stromzuführung, links = Nicht geschaltet, rechts geschaltet
 - Räumliche Trennung von 230V und Niedervoltspannungen auf der Platine
 
Neu 0.23 - P300_Display_IF
 - Platine zum Aufstecken des Displays für die räumlich getrennte Montage von Display zu P300_Arduino_IF
Parts:
- added J15: TFT Display 1, Connector_Molex:Molex_KK-6410-08_08x2.54mm_Straight, symbol P300_Arduino_IF-rescue:Conn_01x08-Connector_Generic
- added J16: TFT Display 2, Connector_Molex:Molex_KK-254_AE-6410-08A_1x08_P2.54mm_Vertical, symbol P300_Arduino_IF-rescue:Conn_01x08-Connector_Generic
Connections:
- net +5V: now also J15.7 (Pin_7)
- net GND: now also J15.6 (Pin_6)
- net PWM_L1: now also R6.2; no longer R5.2
- net PWM_L2: now also R5.2; no longer R6.2
- net Tacho_L1: now also J4.5 (Pin_5); no longer J4.1 (Pin_1)
- net Tacho_L2: now also J4.1 (Pin_1); no longer J4.5 (Pin_5)
- net +3V3: now reaches XA1.3V3 (3.3V)
- net +3V3: now also J15.8 (Pin_8)
- net LCD_RD: now reaches XA1.A0
- net LCD_RD: now also J15.5 (Pin_5)
- net LCD_WR: now reaches XA1.A1
- net LCD_WR: now also J15.4 (Pin_4)
- net LCD_RS: now reaches XA1.A2
- net LCD_RS: now also J15.3 (Pin_3)
- net LCD_CS: now reaches XA1.A3
- net LCD_CS: now also J15.2 (Pin_2)
- net LCD_RST: now reaches XA1.A4
- net LCD_RST: now also J15.1 (Pin_1)
- net LCD_D5: now reaches XA1.D10
- net LCD_D5: now also J16.4 (Pin_4)
- net LCD_D4: now reaches XA1.D11
- net LCD_D4: now also J16.3 (Pin_3)
- net LCD_D3: now reaches XA1.D12
- net LCD_D3: now also J16.2 (Pin_2)
- net LCD_D2: now reaches XA1.D13
- net LCD_D2: now also J16.1 (Pin_1)
- net LCD_D1: now reaches XA1.D6
- net LCD_D1: now also J16.8 (Pin_8)
- net LCD_D0: now reaches XA1.D7
- net LCD_D0: now also J16.7 (Pin_7)
- net LCD_D7: now reaches XA1.D8
- net LCD_D7: now also J16.6 (Pin_6)
- net LCD_D6: now reaches XA1.D9
- net LCD_D6: now also J16.5 (Pin_5)
Other:
- note added: "Lüfter L1 ist Zuluft\nLüfter L2 ist Abluft\n(wegen Belegungskompatibilität \ndes Steckers mit Pluggit ist:\n L2 auf Stecker Pin1-4 und \n L1 auf Stecker Pin5-8)"
- moved on the sheet: J12, J13, J4, R5, R6, U1, U2
